File: tests/fixtures/polcap_rail_correct.kicad_sch (KiCad schematic)
At the start: 3 parts, among them J1 Conn_01x02

Commit message: test: deliberately reverse C1 to prove the Action catches it
Not to be merged. This replaces the correct board with the reversed one so the
self-connectivity workflow has a real defect to find.
Connections:
- net GND: now also C1.1; no longer C1.2
- net VIN: now also C1.2; no longer C1.1
Changed lines of the file:
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@@
     (instances
       (project "SKiDL-Generated"
-        (path "/c2b992a4-58e1-4121-9aad-43cc5fbe9f83"
+        (path "/6bb68f96-1a38-4fe3-9393-666e64f6e1f3"
           (reference "J1")
           (unit 1)))))
@@
     (instances
       (project "SKiDL-Generated"
-        (path "/c2b992a4-58e1-4121-9aad-43cc5fbe9f83"
+        (path "/6bb68f96-1a38-4fe3-9393-666e64f6e1f3"
           (reference "C1")
           (unit 1)))))
@@
     (instances
       (project "SKiDL-Generated"
-        (path "/c2b992a4-58e1-4121-9aad-43cc5fbe9f83"
+        (path "/6bb68f96-1a38-4fe3-9393-666e64f6e1f3"
           (reference "R1")
           (unit 1)))))
@@
           (reference "#PWR001")
           (unit 1)))))
-  (global_label "VIN"
-    (shape bidirectional)
-    (at 144.78 99.06 180)
-    (effects
-      (font
-        (size 1.27 1.27))
-      (justify right))
-)
   (symbol
     (lib_id "power:GND")
-    (at 152.4 99.06 90.0)
+    (at 144.78 99.06 270.0)
     (unit 1)
     (exclude_from_sim yes)
@@
     (fields_autoplaced yes)
     (property "Reference" "#PWR002"
-      (at 152.4 97.79 0)
+      (at 144.78 97.79 0)
       (effects
         (font
@@
         (hide yes)))
     (property "Value" "GND"
-      (at 152.4 95.25 0)
+      (at 144.78 95.25 0)
       (effects
         (font
           (size 1.27 1.27))))
     (property "Footprint" ""
-      (at 152.4 99.06 0)
+      (at 144.78 99.06 0)
       (effects
         (font
@@
         (hide yes)))
     (property "Datasheet" ""
-      (at 152.4 99.06 0)
+      (at 144.78 99.06 0)
       (effects
         (font
@@
   (global_label "VIN"
     (shape bidirectional)
+    (at 152.4 99.06 0)
+    (effects
+      (font
+        (size 1.27 1.27))
+      (justify left))
+)
+  (global_label "VIN"
+    (shape bidirectional)
